File: q605-power-supply.sch (KiCad schematic (older format))
At the start: 3 parts

Commit message: First draft, still missing inverting 5V supply
Parts:
- removed R?: R_US, symbol Device:R_US
- removed U?: ATtiny85V-10PU, Package_DIP:DIP-8_W7.62mm, symbol MCU_Microchip_ATtiny:ATtiny85V-10PU
- added C?: 0.1u, symbol Device:C
- added J? (x2): Screw_Terminal_01x02, symbol Connector:Screw_Terminal_01x02
- added Q? (x2): Q_NPN_CBE, symbol Device:Q_NPN_CBE
- added R? (x3): 10k, symbol Device:R_US
- added R?: 0, symbol Device:R_US
- added R?: 1k, symbol Device:R_US
- added U?: PIC16F18313, Package_DIP:DIP-8_W7.62mm, symbol michel:PIC16F18313-IP
Connections:
- net labels added: +12V, +3V3, +5V, +5VA, -12V, -5V, ATX_PWR_OK, GND, LED_A, LED_K, PWR_LED, PWR_SW, ~ATX_PWR_ON~
- wire segments 0 -> 31
Other:
- moved on the sheet: J?

Commit message: Update q605-power-supply.sch
Parts:
- removed Q?: Q_NPN_CBE, symbol Device:Q_NPN_CBE
- added C?: 0.1u, symbol Device:C
Connections:
- net +5VA: now also C?.1
- net GND: now also C?.2
Changed lines of the file:
@@
 Wire Wire Line
 	7650 3600 7650 3550
-$Comp
-L Device:Q_NPN_CBE Q?
-U 1 1 5F8D6582
-P 9650 1850
-F 0 "Q?" H 9841 1896 50  0000 L CNN
-F 1 "Q_NPN_CBE" H 9841 1805 50  0000 L CNN
-F 2 "" H 9850 1950 50  0001 C CNN
-F 3 "~" H 9650 1850 50  0001 C CNN
-	1    9650 1850
-	1    0    0    -1
-$EndComp
 Text Label 8250 2450 0    50   ~ 0
 ATX_PWR_OK
@@
 Wire Wire Line
 	3650 4650 3600 4650
+$Comp
+L Device:C C?
+U 1 1 5F92DED9
+P 5450 3900
+F 0 "C?" H 5565 3946 50  0000 L CNN
+F 1 "0.1u" H 5565 3855 50  0000 L CNN
+F 2 "" H 5488 3750 50  0001 C CNN
+F 3 "~" H 5450 3900 50  0001 C CNN
+	1    5450 3900
+	1    0    0    -1
+$EndComp
+$Comp
+L power:+5VA #PWR?
+U 1 1 5F92F161
+P 5450 3700
+F 0 "#PWR?" H 5450 3550 50  0001 C CNN
+F 1 "+5VA" H 5465 3873 50  0000 C CNN
+F 2 "" H 5450 3700 50  0001 C CNN
+F 3 "" H 5450 3700 50  0001 C CNN
+	1    5450 3700
+	1    0    0    -1
+$EndComp
+$Comp
+L power:GND #PWR?
+U 1 1 5F92F5EA
+P 5450 4100
+F 0 "#PWR?" H 5450 3850 50  0001 C CNN
+F 1 "GND" H 5455 3927 50  0000 C CNN
+F 2 "" H 5450 4100 50  0001 C CNN
+F 3 "" H 5450 4100 50  0001 C CNN
+	1    5450 4100
+	1    0    0    -1
+$EndComp
+Wire Wire Line
+	5450 3700 5450 3750
+Wire Wire Line
+	5450 4050 5450 4100
 $EndSCHEMATC

Commit message: Finished schematic placement and annotation
Parts:
- added C?: 330n, symbol Device:CP1
- added C?: 1u, symbol Device:CP1
- added J?: Screw_Terminal_01x05, symbol Connector:Screw_Terminal_01x05
- added R?: 10k, symbol Device:R_US
- added U2: MC79M05_TO220, Package_TO_SOT_THT:TO-220-3_Vertical, symbol Regulator_Linear:MC79M05_TO220
- gave numbers to parts that had none: 4
Connections:
- net +12V: now also J?.2 (Pin_2)
- net +5V: now also J?.3 (Pin_3)
- net +5VA: now also R?.2
- net -12V: now also C?.2, U2.2 (VI)
- net -5V: now also C?.2, J?.1 (Pin_1), U2.3 (VO)
- net GND: now also C?.1, C?.1, J?.4 (Pin_4), J?.5 (Pin_5), U2.1 (GND)
- net PWR_LED: now also U1.5 (RA2)
- net ~ATX_PWR_ON~: now also U1.2 (RA5)
- net ~MCLR~: now reaches U1.4 (VPP/~MCLR~/RA3)
- net ~MCLR~: now also R?.1
- net ICSP_CLK: now reaches U1.6 (RA1/ICSPCLK)
- net ICSP_DAT: now reaches U1.7 (RA0/ICSPDAT)
- no-connect marks 0 -> 1
Other:
- moved on the sheet: C?, J1, R?, U1

Commit message: Added programming header and assigned footprints
Parts:
- added J5: Conn_01x06, Connector_PinHeader_2.54mm:PinHeader_1x06_P2.54mm_Vertical, symbol Connector_Generic:Conn_01x06
- C1, C2: renamed from C?; footprint (none) -> Capacitor_THT:C_Disc_D3.0mm_W1.6mm_P2.50mm
- C3, C4: renamed from C?; footprint (none) -> Capacitor_THT:CP_Radial_D4.0mm_P2.00mm
- J1: footprint (none) -> Connector_Molex:Molex_Mini-Fit_Jr_5566-24A_2x12_P4.20mm_Vertical
- J2, J3: footprint (none) -> TerminalBlock_TE-Connectivity:TerminalBlock_TE_282834-2_1x02_P2.54mm_Horizontal
- J4: renamed from J?; footprint (none) -> TerminalBlock_TE-Connectivity:TerminalBlock_TE_282834-5_1x05_P2.54mm_Horizontal
- Q1: renamed from Q?; footprint (none) -> Package_TO_SOT_THT:TO-92
- R1, R2, R3, R4, R5, R6: renamed from R?; footprint (none) -> Resistor_THT:R_Axial_DIN0204_L3.6mm_D1.6mm_P5.08mm_Horizontal
Connections:
- net +5VA: now also J5.2 (Pin_2)
- net GND: now also J5.3 (Pin_3)
- net ICSP_CLK: now also J5.5 (Pin_5)
- net ICSP_DAT: now also J5.4 (Pin_4)
- net ~MCLR~: now also J5.1 (Pin_1)
- no-connect marks 1 -> 2

Commit message: Finished routing
Parts:
- removed Q1: Q_NPN_CBE, Package_TO_SOT_THT:TO-92, symbol Device:Q_NPN_CBE
- added Q1: Q_NPN_EBC, Package_TO_SOT_THT:TO-92, symbol Device:Q_NPN_EBC
- J2, J3: footprint TerminalBlock_TE-Connectivity:TerminalBlock_TE_282834-2_1x02_P2.54mm_Horizontal -> TerminalBlock_RND:TerminalBlock_RND_205-00001_1x02_P5.00mm_Horizontal
- J4: footprint TerminalBlock_TE-Connectivity:TerminalBlock_TE_282834-5_1x05_P2.54mm_Horizontal -> TerminalBlock_RND:TerminalBlock_RND_205-00004_1x05_P5.00mm_Horizontal
Connections:
- net ATX_PWR_OK: now also U1.5 (RA2)
- net GND: now also Q1.1 (E)
- net LED_K: now also Q1.3 (C)
- net PWR_LED: now also U1.3 (RA4); no longer U1.5 (RA2)
- net at R4.2: now also Q1.2 (B)
- net +3V3: no longer names the net of J1.1 (+3.3V), J1.12 (+3.3V), J1.13 (+3.3V), J1.2 (+3.3V)
Other:
- moved on the sheet: C1, C2, C3, C4, J1, J2, J3, J4, J5, R1, R2, R3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
