File: pcb/q605-power-supply.sch (KiCad schematic (older format))
At the start: 18 parts, among them J1 ATX-24, J2 Screw_Terminal_01x02, J3 Screw_Terminal_01x02, J4 Screw_Terminal_01x05, J5 Conn_01x06, Q1 Q_NPN_EBC, U1 PIC16F18313, U2 MC79M05_TO220

Commit message: Moving to PCB folder
Parts:
- added R7: 10k, Resistor_THT:R_Axial_DIN0204_L3.6mm_D1.6mm_P5.08mm_Horizontal, symbol Device:R_US
Connections:
- net ATX_PWR_OK: now also R7.2; no longer U1.5 (RA2)
- net ICSP_DAT: now also R7.1
- net PWR_SW: now also U1.5 (RA2)
Other:
- note added: "-12V to -5V LDO"
- note added: "24-pin ATX Connector"
- note added: "Microcontroller + Programming"
- note added: "Q605 PSU Output + Power Switch + Power LED"
- moved on the sheet: C3, C4, J5, U2
